Commit message: Fixed the gazebo sim issues.

File: models/urdf/fastbot_body.xacro (robot description, xacro)
@@ -186,9 +186,9 @@
     </joint>
     <!-- Link lslidar_n10 -->
-    <link name="${robot_name}_n10_v2">
+    <link name="${robot_name}_lidar">
         <inertial>
             <origin xyz="0 0 0" rpy="0 0 0"/>
             <mass value="0.05"/>
-            <inertia ixx="1e-09" ixy="0" ixz="0" iyy="1e-09" iyz="0" izz="1e-09"/>
+            <inertia ixx="0.0001" ixy="0" ixz="0" iyy="0.0001" iyz="0" izz="0.0002"/>
         </inertial>
         <!-- Part lslidar_n10 -->
@@ -211,7 +211,7 @@
     <!-- Joint from fastbot_chassis to lslidar_n10 -->
     <joint name="${robot_name}_lidar" type="fixed">
-        <origin xyz="-0.0166657 -0.00914257 0.111345" rpy="3.14159 1.13983e-46 -3.14159"/>
-        <parent link="${robot_name}_base_link"/>
-        <child link="${robot_name}_n10_v2"/>
+        <origin xyz="-0.0166657 0 0.112" rpy="3.14159 1.13983e-46 -3.14159"/>
+        <parent link="${robot_name}_base_link"/>
+        <child link="${robot_name}_lidar"/>
         <axis xyz="0 0 1"/>
     </joint>
@@ -242,5 +242,5 @@
     <!-- Joint from fastbot_chassis to raspicam -->
     <joint name="${robot_name}_camera" type="fixed">
-        <origin xyz="0.00783428 -0.0661426 0.100995" rpy="-1.5708 1.14468e-45 6.41848e-15"/>
+        <origin xyz="0.00783428 -0.0661426 0.100995" rpy="0 0 -1.5708"/>
         <parent link="${robot_name}_base_link"/>
         <child link="${robot_name}_camera"/>
